Commit message: Includes two boxes and two arms

File: assets/cube_blue.urdf (robot description, URDF)
Before this commit: robot cube.urdf, 1 links, 0 joints
Links:
- link cube: geometry collision box size=0.06 0.06 0.06; visual box size=0.06 0.06 0.06

File: assets/cube_red.urdf (robot description, URDF)
Before this commit: robot cube.urdf, 1 links, 0 joints
Links:
- link cube: geometry collision box size=0.06 0.06 0.06; visual box size=0.06 0.06 0.06
